File: Kicad/Motherboard/8088 PCB.sch (KiCad schematic (older format))
At the start: 78 parts, among them J1 Bus_ISA_8bit, J2 Mini-DIN-6, J3 SPK, J4 CS7, SW1 RESET, U1 8088, U10 8237, U11 74LS573, U12 74LS139, U13 AS6C4008, U14 AS6C1008, U15 27C512, U16 74LS138, U17 8284, U18 74LS74, U19 W83C42P, U2 74LS573, U20 74LS07, U21 74LS04, U22 8284, U23 74LS245, U24 74LS573, U25 74LS126, U26 74LS125, U3 74LS573, U4 74LS245, U5 8254, U6 8259, U7 74LS670, U8 74LS257, U9 27C512, Y1 14.31818, Y2 CRYSTAL

Commit message: Update IRQ 1 pin
Parts:
- added J5: IRQ 1, Connector_PinHeader_2.54mm:PinHeader_1x01_P2.54mm_Vertical, symbol Connector_Generic:Conn_01x01
Connections:
- net IRQ1: now also J5.1 (Pin_1)
Changed lines of the file:
@@
 Text Label 3750 6725 0    50   ~ 0
 5+
+$Comp
+L Connector_Generic:Conn_01x01 J5
+U 1 1 66552FD8
+P 12025 975
+F 0 "J5" H 12105 1017 50  0000 L CNN
+F 1 "IRQ 1" H 12105 926 50  0000 L CNN
+F 2 "Connector_PinHeader_2.54mm:PinHeader_1x01_P2.54mm_Vertical" H 12025 975 50  0001 C CNN
+F 3 "~" H 12025 975 50  0001 C CNN
+	1    12025 975
+	1    0    0    -1
+$EndComp
+Text Label 11825 975  2    50   ~ 0
+IRQ1
 $EndSCHEMATC

Commit message: Update
Parts:
- U11, U2, U24, U3: value 74LS573 -> 74*573
- U12: value 74LS139 -> 74*139
- U16: value 74LS138 -> 74*138
- U18: value 74LS74 -> 74*74
- U19: value W83C42P -> 82C42
- U20: value 74LS07 -> 74*07
- U21: value 74LS04 -> 74*04
- U23, U4: value 74LS245 -> 74*245
- U25: value 74LS126 -> 74*126
- U26: value 74LS125 -> 74*125
- U7: value 74LS670 -> 74*670
- U8: value 74LS257 -> 74*257
Changed lines of the file:
@@
 P 4625 1900
 F 0 "U2" H 4625 2881 50  0000 C CNN
-F 1 "74LS573" H 4625 2790 50  0000 C CNN
+F 1 "74*573" H 4625 2790 50  0000 C CNN
 F 2 "Package_DIP:DIP-20_W7.62mm" H 4625 1900 50  0001 C CNN
 F 3 "74xx/74hc573.pdf" H 4625 1900 50  0001 C CNN
@@
 P 4350 4100
 F 0 "U3" H 4350 5081 50  0000 C CNN
-F 1 "74LS573" H 4350 4990 50  0000 C CNN
+F 1 "74*573" H 4350 4990 50  0000 C CNN
 F 2 "Package_DIP:DIP-20_W7.62mm" H 4350 4100 50  0001 C CNN
 F 3 "74xx/74hc573.pdf" H 4350 4100 50  0001 C CNN
@@
 P 4625 6450
 F 0 "U4" H 4625 7431 50  0000 C CNN
-F 1 "74LS245" H 4625 7340 50  0000 C CNN
+F 1 "74*245" H 4625 7340 50  0000 C CNN
 F 2 "Package_DIP:DIP-20_W7.62mm" H 4625 6450 50  0001 C CNN
 F 3 "http://www.ti.com/lit/gpn/sn74LS245" H 4625 6450 50  0001 C CNN
@@
 P 1925 6825
 F 0 "U8" H 1925 7906 50  0000 C CNN
-F 1 "74LS257" H 1925 7815 50  0000 C CNN
+F 1 "74*257" H 1925 7815 50  0000 C CNN
 F 2 "Package_DIP:DIP-16_W7.62mm" H 1925 6825 50  0001 C CNN
 F 3 "http://www.ti.com/lit/gpn/sn74LS257" H 1925 6825 50  0001 C CNN
@@
 P 18675 2025
 F 0 "U7" H 18675 3006 50  0000 C CNN
-F 1 "74LS670" H 18675 2915 50  0000 C CNN
+F 1 "74*670" H 18675 2915 50  0000 C CNN
 F 2 "Package_DIP:DIP-16_W7.62mm" H 18675 2025 50  0001 C CNN
 F 3 "http://www.ti.com/lit/gpn/sn74LS670" H 18675 2025 50  0001 C CNN
@@
 P 18650 4225
 F 0 "U11" H 18650 5206 50  0000 C CNN
-F 1 "74LS573" H 18650 5115 50  0000 C CNN
+F 1 "74*573" H 18650 5115 50  0000 C CNN
 F 2 "Package_DIP:DIP-20_W7.62mm" H 18650 4225 50  0001 C CNN
 F 3 "74xx/74hc573.pdf" H 18650 4225 50  0001 C CNN
@@
 P 1575 10000
 F 0 "U12" H 1575 10367 50  0000 C CNN
-F 1 "74LS139" H 1575 10276 50  0000 C CNN
+F 1 "74*139" H 1575 10276 50  0000 C CNN
 F 2 "Package_DIP:DIP-16_W7.62mm" H 1575 10000 50  0001 C CNN
 F 3 "http://www.ti.com/lit/ds/symlink/sn74ls139a.pdf" H 1575 10000 50  0001 C CNN
@@
 P 1575 10500
 F 0 "U12" H 1575 10867 50  0000 C CNN
-F 1 "74LS139" H 1575 10776 50  0000 C CNN
+F 1 "74*139" H 1575 10776 50  0000 C CNN
 F 2 "Package_DIP:DIP-16_W7.62mm" H 1575 10500 50  0001 C CNN
 F 3 "http://www.ti.com/lit/ds/symlink/sn74ls139a.pdf" H 1575 10500 50  0001 C CNN
@@
 P 1575 11000
 F 0 "U12" V 1208 11000 50  0000 C CNN
-F 1 "74LS139" V 1299 11000 50  0000 C CNN
+F 1 "74*139" V 1299 11000 50  0000 C CNN
 F 2 "Package_DIP:DIP-16_W7.62mm" H 1575 11000 50  0001 C CNN
 F 3 "http://www.ti.com/lit/ds/symlink/sn74ls139a.pdf" H 1575 11000 50  0001 C CNN
@@
 P 3625 10550
 F 0 "U16" H 3625 11331 50  0000 C CNN
-F 1 "74LS138" H 3625 11240 50  0000 C CNN
+F 1 "74*138" H 3625 11240 50  0000 C CNN
 F 2 "Package_DIP:DIP-16_W7.62mm" H 3625 10550 50  0001 C CNN
 F 3 "http://www.ti.com/lit/gpn/sn74LS138" H 3625 10550 50  0001 C CNN
@@
 P 16525 6125
 F 0 "U19" H 16525 6190 50  0000 C CNN
-F 1 "W83C42P" H 16525 6099 50  0000 C CNN
+F 1 "82C42" H 16525 6099 50  0000 C CNN
 F 2 "Package_LCC:PLCC-44_THT-Socket" H 16525 6125 50  0001 C CNN
 F 3 "" H 16525 6125 50  0001 C CNN
@@
 P 16200 11250
 F 0 "U18" H 16200 11731 50  0000 C CNN
-F 1 "74LS74" H 16200 11640 50  0000 C CNN
+F 1 "74*74" H 16200 11640 50  0000 C CNN
 F 2 "Package_DIP:DIP-14_W7.62mm" H 16200 11250 50  0001 C CNN
 F 3 "74xx/74hc_hct74.pdf" H 16200 11250 50  0001 C CNN
@@
 P 16200 11975
 F 0 "U18" H 16200 12456 50  0000 C CNN
-F 1 "74LS74" H 16200 12365 50  0000 C CNN
+F 1 "74*74" H 16200 12365 50  0000 C CNN
 F 2 "Package_DIP:DIP-14_W7.62mm" H 16200 11975 50  0001 C CNN
 F 3 "74xx/74hc_hct74.pdf" H 16200 11975 50  0001 C CNN
@@
 P 16225 12750
 F 0 "U18" V 15858 12750 50  0000 C CNN
-F 1 "74LS74" V 15949 12750 50  0000 C CNN
+F 1 "74*74" V 15949 12750 50  0000 C CNN
 F 2 "Package_DIP:DIP-14_W7.62mm" H 16225 12750 50  0001 C CNN
 F 3 "74xx/74hc_hct74.pdf" H 16225 12750 50  0001 C CNN
@@
 P 18100 6300
 F 0 "U20" H 18100 6617 50  0000 C CNN
-F 1 "74LS07" H 18100 6526 50  0000 C CNN
+F 1 "74*07" H 18100 6526 50  0000 C CNN
 F 2 "Package_DIP:DIP-14_W7.62mm" H 18100 6300 50  0001 C CNN
 F 3 "www.ti.com/lit/ds/symlink/sn74ls07.pdf" H 18100 6300 50  0001 C CNN
@@
 P 18100 6775
 F 0 "U20" H 18100 7092 50  0000 C CNN
-F 1 "74LS07" H 18100 7001 50  0000 C CNN
+F 1 "74*07" H 18100 7001 50  0000 C CNN
 F 2 "Package_DIP:DIP-14_W7.62mm" H 18100 6775 50  0001 C CNN
 F 3 "www.ti.com/lit/ds/symlink/sn74ls07.pdf" H 18100 6775 50  0001 C CNN
@@
 P 18100 7450
 F 0 "U20" V 17733 7450 50  0000 C CNN
-F 1 "74LS07" V 17824 7450 50  0000 C CNN
+F 1 "74*07" V 17824 7450 50  0000 C CNN
 F 2 "Package_DIP:DIP-14_W7.62mm" H 18100 7450 50  0001 C CNN
 F 3 "www.ti.com/lit/ds/symlink/sn74ls07.pdf" H 18100 7450 50  0001 C CNN
@@
 P 14250 6150
 F 0 "U21" H 14250 6467 50  0000 C CNN
-F 1 "74LS04" H 14250 6376 50  0000 C CNN
+F 1 "74*04" H 14250 6376 50  0000 C CNN
 F 2 "Package_DIP:DIP-14_W7.62mm" H 14250 6150 50  0001 C CNN
 F 3 "http://www.ti.com/lit/gpn/sn74LS04" H 14250 6150 50  0001 C CNN
@@
 P 14250 6525
 F 0 "U21" H 14250 6842 50  0000 C CNN
-F 1 "74LS04" H 14250 6751 50  0000 C CNN
+F 1 "74*04" H 14250 6751 50  0000 C CNN
 F 2 "Package_DIP:DIP-14_W7.62mm" H 14250 6525 50  0001 C CNN
 F 3 "http://www.ti.com/lit/gpn/sn74LS04" H 14250 6525 50  0001 C CNN
@@
 P 14250 6925
 F 0 "U21" H 14250 7242 50  0000 C CNN
-F 1 "74LS04" H 14250 7151 50  0000 C CNN
+F 1 "74*04" H 14250 7151 50  0000 C CNN
 F 2 "Package_DIP:DIP-14_W7.62mm" H 14250 6925 50  0001 C CNN
 F 3 "http://www.ti.com/lit/gpn/sn74LS04" H 14250 6925 50  0001 C CNN
@@
 P 14250 7300
 F 0 "U21" H 14250 7617 50  0000 C CNN
-F 1 "74LS04" H 14250 7526 50  0000 C CNN
+F 1 "74*04" H 14250 7526 50  0000 C CNN
 F 2 "Package_DIP:DIP-14_W7.62mm" H 14250 7300 50  0001 C CNN
 F 3 "http://www.ti.com/lit/gpn/sn74LS04" H 14250 7300 50  0001 C CNN
@@
 P 14250 8900
 F 0 "U21" V 13883 8900 50  0000 C CNN
-F 1 "74LS04" V 13974 8900 50  0000 C CNN
+F 1 "74*04" V 13974 8900 50  0000 C CNN
 F 2 "Package_DIP:DIP-14_W7.62mm" H 14250 8900 50  0001 C CNN
 F 3 "http://www.ti.com/lit/gpn/sn74LS04" H 14250 8900 50  0001 C CNN
@@
 P 7725 6350
 F 0 "U23" H 7725 7331 50  0000 C CNN
-F 1 "74LS245" H 7725 7240 50  0000 C CNN
+F 1 "74*245" H 7725 7240 50  0000 C CNN
 F 2 "Package_DIP:DIP-20_W7.62mm" H 7725 6350 50  0001 C CNN
 F 3 "http://www.ti.com/lit/gpn/sn74LS245" H 7725 6350 50  0001 C CNN
@@
 P 9500 6400
 F 0 "U24" H 9500 7381 50  0000 C CNN
-F 1 "74LS573" H 9500 7290 50  0000 C CNN
+F 1 "74*573" H 9500 7290 50  0000 C CNN
 F 2 "Package_DIP:DIP-20_W7.62mm" H 9500 6400 50  0001 C CNN
 F 3 "74xx/74hc573.pdf" H 9500 6400 50  0001 C CNN
@@
 P 11400 6000
 F 0 "U26" H 11400 6317 50  0000 C CNN
-F 1 "74LS125" H 11400 6226 50  0000 C CNN
+F 1 "74*125" H 11400 6226 50  0000 C CNN
 F 2 "Package_DIP:DIP-14_W7.62mm" H 11400 6000 50  0001 C CNN
 F 3 "http://www.ti.com/lit/gpn/sn74LS126" H 11400 6000 50  0001 C CNN
@@
 P 11400 6375
 F 0 "U26" H 11400 6692 50  0000 C CNN
-F 1 "74LS125" H 11400 6601 50  0000 C CNN
+F 1 "74*125" H 11400 6601 50  0000 C CNN
 F 2 "Package_DIP:DIP-14_W7.62mm" H 11400 6375 50  0001 C CNN
 F 3 "http://www.ti.com/lit/gpn/sn74LS126" H 11400 6375 50  0001 C CNN
@@
 P 11325 7100
 F 0 "U26" V 10958 7100 50  0000 C CNN
-F 1 "74LS125" V 11049 7100 50  0000 C CNN
+F 1 "74*125" V 11049 7100 50  0000 C CNN
 F 2 "Package_DIP:DIP-14_W7.62mm" H 11325 7100 50  0001 C CNN
 F 3 "http://www.ti.com/lit/gpn/sn74LS126" H 11325 7100 50  0001 C CNN
@@
 P 11375 7750
 F 0 "U25" H 11375 8067 50  0000 C CNN
-F 1 "74LS126" H 11375 7976 50  0000 C CNN
+F 1 "74*126" H 11375 7976 50  0000 C CNN
 F 2 "Package_DIP:DIP-14_W7.62mm" H 11375 7750 50  0001 C CNN
 F 3 "http://www.ti.com/lit/gpn/sn74LS126" H 11375 7750 50  0001 C CNN
@@
 P 11350 8375
 F 0 "U25" H 11350 8692 50  0000 C CNN
-F 1 "74LS126" H 11350 8601 50  0000 C CNN
+F 1 "74*126" H 11350 8601 50  0000 C CNN
 F 2 "Package_DIP:DIP-14_W7.62mm" H 11350 8375 50  0001 C CNN
 F 3 "http://www.ti.com/lit/gpn/sn74LS126" H 11350 8375 50  0001 C CNN
@@
 P 11375 9175
 F 0 "U25" V 11008 9175 50  0000 C CNN
-F 1 "74LS126" V 11099 9175 50  0000 C CNN
+F 1 "74*126" V 11099 9175 50  0000 C CNN
 F 2 "Package_DIP:DIP-14_W7.62mm" H 11375 9175 50  0001 C CNN
 F 3 "http://www.ti.com/lit/gpn/sn74LS126" H 11375 9175 50  0001 C CNN
@@
 P 14250 7700
 F 0 "U21" H 14250 8017 50  0000 C CNN
-F 1 "74LS04" H 14250 7926 50  0000 C CNN
+F 1 "74*04" H 14250 7926 50  0000 C CNN
 F 2 "Package_DIP:DIP-14_W7.62mm" H 14250 7700 50  0001 C CNN
 F 3 "http://www.ti.com/lit/gpn/sn74LS04" H 14250 7700 50  0001 C CNN
@@
 P 11975 6750
 F 0 "U26" H 11975 7067 50  0000 C CNN
-F 1 "74LS125" H 11975 6976 50  0000 C CNN
+F 1 "74*125" H 11975 6976 50  0000 C CNN
 F 2 "Package_DIP:DIP-14_W7.62mm" H 11975 6750 50  0001 C CNN
 F 3 "http://www.ti.com/lit/gpn/sn74LS126" H 11975 6750 50  0001 C CNN
@@
 P 14275 8200
 F 0 "U21" H 14275 8517 50  0000 C CNN
-F 1 "74LS04" H 14275 8426 50  0000 C CNN
+F 1 "74*04" H 14275 8426 50  0000 C CNN
 F 2 "Package_DIP:DIP-14_W7.62mm" H 14275 8200 50  0001 C CNN
 F 3 "http://www.ti.com/lit/gpn/sn74LS04" H 14275 8200 50  0001 C CNN
